File: moarPWR/USB_C.sch (KiCad schematic (older format))
At the start: 0 parts

Commit message: Updated part numbers in USB and display control. Added 7 Segment displays and driver.
Parts:
- added J?: USB_C_Receptacle, symbol Connector:USB_C_Receptacle
Changed lines of the file:
@@
 $Descr A4 11693 8268
 encoding utf-8
-Sheet 6 5
+Sheet 5 5
 Title ""
 Date ""
@@
 Comment4 ""
 $EndDescr
+$Comp
+L Connector:USB_C_Receptacle J?
+U 1 1 5B8195C7
+P 9750 3850
+F 0 "J?" H 9855 5417 50  0000 C CNN
+F 1 "USB_C_Receptacle" H 9855 5326 50  0000 C CNN
+F 2 "" H 9900 3850 50  0001 C CNN
+F 3 "http://www.usb.org/developers/docs/usb_31_033017.zip" H 9900 3850 50  0001 C CNN
+	1    9750 3850
+	-1   0    0    -1
+$EndComp
 $EndSCHEMATC
