File: moarPWR/5V_to_USB.sch (KiCad schematic (older format))
At the start: 0 parts

Commit message: Added port controller and power switch for 5V USB channels
Parts:
- added C? (x2): CP1, symbol Device:CP1
- added C?: C, symbol Device:C
- added C? (x2): 0.22uF, symbol Device:C
- added J? (x2): USB_A, symbol Connector:USB_A
- added R?: 25.5K, symbol Device:R
- added R? (x2): R, symbol Device:R
- added U?: TPS2513A, Package_TO_SOT_SMD:SOT-23-6, symbol Interface_USB:TPS2513A
- added U?: TPS2561A, Package_SON:VSON-10-1EP_3x3mm_P0.5mm_EP1.65x2.4mm_ThermalVias, symbol Interface_USB:TPS2561
Connections:
- net labels added: 5VIN, GND, USB_1_SUPPLY, USB_2_SUPPLY, ~FAULT1, ~FAULT2
- wire segments 0 -> 59
Other:
- note added: "SUPPLY_CAP\n"
- note added: "USB_1"
- note added: "USB_2"

Commit message: Updated part numbers in USB and display control. Added 7 Segment displays and driver.
Parts:
- removed C?: CP1, symbol Device:CP1
- removed C?: 0.22uF, symbol Device:C
- removed R?: R, symbol Device:R
- added C?: .1uF, Capacitors_SMD:C_0805_HandSoldering, symbol Device:C
- added C?: 0.22uF, Capacitors_SMD:C_0805_HandSoldering, symbol Device:C
- added C?: CP1, Capacitors_SMD:CP_Elec_6.3x5.8, symbol Device:CP1
- added R?: 100k, Resistors_SMD:R_0805_HandSoldering, symbol Device:R
- C?: footprint (none) -> Capacitors_SMD:CP_Elec_6.3x5.8; Manufacturer (none) -> Nichicon; Manufacturer P/N (none) -> UWT1A151MCL1GS; Vendor P/N (none) -> 493-2166-1-ND
- C?: value C -> 10uF; footprint (none) -> Capacitors_SMD:C_0805_HandSoldering; Manufacturer (none) -> Samsung; Manufacturer P/N (none) -> CL21A106KQCLNNC; Vendor (none) -> Digi-Key; Vendor P/N (none) -> 1276-2404-1-ND
- C?: footprint (none) -> Capacitors_SMD:C_0805_HandSoldering; Manufacturer (none) -> Samsung; Manufacturer P/N (none) -> CL21A226KQCLRNC; Vendor (none) -> Digi-Key; Vendor P/N (none) -> 1276-6687-1-ND
- R?: footprint (none) -> Resistors_SMD:R_0805_HandSoldering; Manufacturer (none) -> Yageo; Manufacturer P/N (none) -> RC0805FR-0725K5L; Vendor (none) -> Digi-Key; Vendor P/N (none) -> 311-25.5KCRCT-ND
- R?: value R -> 100k; footprint (none) -> Resistors_SMD:R_0805_HandSoldering; Manufacturer (none) -> Panasonic; Manufacturer P/N (none) -> ERA-6AEB104V; Vendor (none) -> Digi-Key; Vendor P/N (none) -> P100KDACT-ND
Connections:
- net labels added: +5V
- net labels removed: 5VIN
- wire segments 59 -> 65

Commit message: Added MSP and current sense amplifier
Parts:
- added C?: .1uF, Capacitors_SMD:C_0805_HandSoldering, symbol Device:C
- added R? (x2): R, symbol Device:R
- added U?: INA2180, symbol MERKL_LIB:INA2180
Connections:
- net labels added: C_SENSE_0, C_SENSE_1
- wire segments 65 -> 83
Other:
- moved on the sheet: U?

Commit message: Added I2C
Changed lines of the file:
@@
 L MERKL_LIB:INA2180 U?
 U 1 1 5C6282FC
-P 2700 6350
-F 0 "U?" H 2950 6800 50  0000 C CNN
-F 1 "INA2180" H 2900 5850 50  0000 C CNN
-F 2 "" H 2650 6500 50  0001 C CNN
-F 3 "" H 2650 6500 50  0001 C CNN
-	1    2700 6350
+P 8550 1950
+F 0 "U?" H 8800 2400 50  0000 C CNN
+F 1 "INA2180" H 8750 1450 50  0000 C CNN
+F 2 "" H 8500 2100 50  0001 C CNN
+F 3 "" H 8500 2100 50  0001 C CNN
+	1    8550 1950
 	1    0    0    -1
 $EndComp
@@
 L Device:R R?
 U 1 1 5C62DE0F
-P 1500 6200
-F 0 "R?" H 1570 6246 50  0000 L CNN
-F 1 "R" H 1570 6155 50  0000 L CNN
-F 2 "" V 1430 6200 50  0001 C CNN
-F 3 "~" H 1500 6200 50  0001 C CNN
-	1    1500 6200
+P 7350 1800
+F 0 "R?" H 7420 1846 50  0000 L CNN
+F 1 "R" H 7420 1755 50  0000 L CNN
+F 2 "" V 7280 1800 50  0001 C CNN
+F 3 "~" H 7350 1800 50  0001 C CNN
+	1    7350 1800
 	1    0    0    -1
 $EndComp
@@
 L Device:R R?
 U 1 1 5C62DEA4
-P 1500 6600
-F 0 "R?" H 1570 6646 50  0000 L CNN
-F 1 "R" H 1570 6555 50  0000 L CNN
-F 2 "" V 1430 6600 50  0001 C CNN
-F 3 "~" H 1500 6600 50  0001 C CNN
-	1    1500 6600
+P 7350 2200
+F 0 "R?" H 7420 2246 50  0000 L CNN
+F 1 "R" H 7420 2155 50  0000 L CNN
+F 2 "" V 7280 2200 50  0001 C CNN
+F 3 "~" H 7350 2200 50  0001 C CNN
+	1    7350 2200
 	1    0    0    -1
 $EndComp
-Text Label 1150 6350 2    50   ~ 0
+Text Label 7000 1950 2    50   ~ 0
 USB_1_SUPPLY
-Text Label 1150 6450 2    50   ~ 0
+Text Label 7000 2050 2    50   ~ 0
 USB_2_SUPPLY
 Wire Wire Line
-	2200 6200 1900 6200
+	8050 1800 7750 1800
 Wire Wire Line
-	1900 6200 1900 6050
+	7750 1800 7750 1650
 Wire Wire Line
-	1900 6050 1500 6050
+	7750 1650 7350 1650
 Wire Wire Line
-	2200 6300 1900 6300
+	8050 1900 7750 1900
 Wire Wire Line
-	1900 6300 1900 6350
+	7750 1900 7750 1950
 Wire Wire Line
-	1900 6350 1500 6350
-Connection ~ 1500 6350
+	7750 1950 7350 1950
+Connection ~ 7350 1950
 Wire Wire Line
-	1500 6350 1150 6350
+	7350 1950 7000 1950
 Wire Wire Line
-	2200 6400 1750 6400
+	8050 2000 7600 2000
 Wire Wire Line
-	1750 6400 1750 6450
+	7600 2000 7600 2050
 Wire Wire Line
-	1750 6450 1500 6450
-Connection ~ 1500 6450
+	7600 2050 7350 2050
+Connection ~ 7350 2050
 Wire Wire Line
-	1150 6450 1500 6450
+	7000 2050 7350 2050
 Wire Wire Line
-	2200 6500 2200 6750
+	8050 2100 8050 2350
 Wire Wire Line
-	2200 6750 1500 6750
-Text HLabel 3250 6200 2    50   Input ~ 0
+	8050 2350 7350 2350
+Text HLabel 9100 1800 2    50   Input ~ 0
 C_SENSE_0
-Text HLabel 3250 6300 2    50   Input ~ 0
+Text HLabel 9100 1900 2    50   Input ~ 0
 C_SENSE_1
 $Comp
 L power:+5V #PWR?
 U 1 1 5C63D8A5
-P 2700 5450
-F 0 "#PWR?" H 2700 5300 50  0001 C CNN
-F 1 "+5V" H 2715 5623 50  0000 C CNN
-F 2 "" H 2700 5450 50  0001 C CNN
-F 3 "" H 2700 5450 50  0001 C CNN
-	1    2700 5450
+P 8550 1050
+F 0 "#PWR?" H 8550 900 50  0001 C CNN
+F 1 "+5V" H 8565 1223 50  0000 C CNN
+F 2 "" H 8550 1050 50  0001 C CNN
+F 3 "" H 8550 1050 50  0001 C CNN
+	1    8550 1050
 	1    0    0    -1
 $EndComp
 Wire Wire Line
-	2700 5450 2700 5500
+	8550 1050 8550 1100
 $Comp
 L power:GND #PWR?
 U 1 1 5C63F916
-P 2700 7050
-F 0 "#PWR?" H 2700 6800 50  0001 C CNN
-F 1 "GND" H 2705 6877 50  0000 C CNN
-F 2 "" H 2700 7050 50  0001 C CNN
-F 3 "" H 2700 7050 50  0001 C CNN
-	1    2700 7050
+P 8550 2650
+F 0 "#PWR?" H 8550 2400 50  0001 C CNN
+F 1 "GND" H 8555 2477 50  0000 C CNN
+F 2 "" H 8550 2650 50  0001 C CNN
+F 3 "" H 8550 2650 50  0001 C CNN
+	1    8550 2650
 	1    0    0    -1
 $EndComp
 Wire Wire Line
-	2700 7000 2700 7050
+	8550 2600 8550 2650
 $Comp
 L Device:C C?
 U 1 1 5C6419CB
-P 3300 5650
+P 9150 1250
 AR Path="/5BA57DA6/5C6419CB" Ref="C?"  Part="1"
 AR Path="/5B5E9C4D/5C6419CB" Ref="C?"  Part="1"
-F 0 "C?" H 3415 5696 50  0000 L CNN
-F 1 ".1uF" H 3415 5605 50  0000 L CNN
-F 2 "Capacitors_SMD:C_0805_HandSoldering" H 3338 5500 50  0001 C CNN
-F 3 "~" H 3300 5650 50  0001 C CNN
-F 4 "KEMET" H 3300 5650 50  0001 C CNN "Manufacturer"
-F 5 "C0805X104K4RACTU" H 3300 5650 50  0001 C CNN "Manufacturer P/N"
-F 6 "Digi-Key" H 3300 5650 50  0001 C CNN "Vendor"
-F 7 "399-5331-1-ND" H 3300 5650 50  0001 C CNN "Vendor P/N"
-	1    3300 5650
+F 0 "C?" H 9265 1296 50  0000 L CNN
+F 1 ".1uF" H 9265 1205 50  0000 L CNN
+F 2 "Capacitors_SMD:C_0805_HandSoldering" H 9188 1100 50  0001 C CNN
+F 3 "~" H 9150 1250 50  0001 C CNN
+F 4 "KEMET" H 9150 1250 50  0001 C CNN "Manufacturer"
+F 5 "C0805X104K4RACTU" H 9150 1250 50  0001 C CNN "Manufacturer P/N"
+F 6 "Digi-Key" H 9150 1250 50  0001 C CNN "Vendor"
+F 7 "399-5331-1-ND" H 9150 1250 50  0001 C CNN "Vendor P/N"
+	1    9150 1250
 	1    0    0    -1
 $EndComp
@@
 L power:GND #PWR?
 U 1 1 5C641AB2
-P 3300 5850
-F 0 "#PWR?" H 3300 5600 50  0001 C CNN
-F 1 "GND" H 3305 5677 50  0000 C CNN
-F 2 "" H 3300 5850 50  0001 C CNN
-F 3 "" H 3300 5850 50  0001 C CNN
-	1    3300 5850
+P 9150 1450
+F 0 "#PWR?" H 9150 1200 50  0001 C CNN
+F 1 "GND" H 9155 1277 50  0000 C CNN
+F 2 "" H 9150 1450 50  0001 C CNN
+F 3 "" H 9150 1450 50  0001 C CNN
+	1    9150 1450
 	1    0    0    -1
 $EndComp
 Wire Wire Line
-	3300 5800 3300 5850
+	9150 1400 9150 1450
 Wire Wire Line
-	3300 5500 2700 5500
-Connection ~ 2700 5500
+	9150 1100 8550 1100
+Connection ~ 8550 1100
 Wire Wire Line
-	2700 5500 2700 5750
+	8550 1100 8550 1350
 $EndSCHEMATC
